Commit message: RGB-D 카메라를 통한 local_costmap에 cost 반영 성공

File: limbo/src/limbo_description/urdf/limbo.gazebo.xacro (robot description, xacro)
@@ -52,48 +52,68 @@
   </gazebo>
   <!-- ================================ -->
-<!-- Livox MID-360 Simulation        -->
-<!-- ================================ -->
-<gazebo reference="mid360_link">
-  <sensor name="mid360_sensor" type="gpu_lidar">
-    <topic>mid360</topic>
-    <gz_frame_id>mid360_link</gz_frame_id>
-    <!-- 실제 MID-360의 일반 frame rate -->
-    <update_rate>10</update_rate>
-    <lidar>
-      <scan>
-        <!-- 360 degree horizontal FOV -->
-        <horizontal>
-          <!--
-            360 samples = 약 1도 간격
-            SLAM/Nav 테스트용으로 충분한 초기값
-          -->
-          <samples>720</samples>
-          <resolution>1</resolution>
-          <min_angle>-3.141592653589793</min_angle>
-          <max_angle>3.141592653589793</max_angle>
-        </horizontal>
-        <!-- MID-360 vertical FOV: -7 ~ +52 degrees -->
-        <vertical>
-          <samples>60</samples>
-          <resolution>1</resolution>
-          <!-- -7 deg -->
-          <min_angle>-0.1221730476</min_angle>
-          <!-- +52 deg -->
-          <max_angle>0.9075712110</max_angle>
-        </vertical>
-      </scan>
-      <range>
-        <!-- 실제 MID-360 최소 측정거리 -->
-        <min>0.10</min>
-        <!-- 10% reflectivity 기준 -->
-        <max>40.0</max>
-        <!-- 거리 resolution은 simulation 설정값 -->
-        <resolution>0.01</resolution>
-      </range>
-    </lidar>
-    <always_on>true</always_on>
-    <!-- Gazebo에서 광선을 눈으로 보고 싶으면 true -->
-    <visualize>true</visualize>
-  </sensor>
-</gazebo>
+  <!-- Livox MID-360 Simulation         -->
+  <!-- ================================ -->
+  <!--
+    The sensor is attached to mid360_link. Its physical position is defined
+    by mid360_joint in limbo.urdf.xacro, so no Gazebo-side XYZ change is
+    required when the LiDAR mount moves.
+  -->
+  <gazebo reference="mid360_link">
+    <sensor name="mid360_sensor" type="gpu_lidar">
+      <topic>mid360</topic>
+      <gz_frame_id>mid360_link</gz_frame_id>
+      <!-- MID-360 general frame rate -->
+      <update_rate>10</update_rate>
+      <lidar>
+        <scan>
+          <!-- 360 degree horizontal FOV -->
+          <horizontal>
+            <samples>720</samples>
+            <resolution>1</resolution>
+            <min_angle>-3.141592653589793</min_angle>
+            <max_angle>3.141592653589793</max_angle>
+          </horizontal>
+          <!-- MID-360 vertical FOV: -7 ~ +52 degrees -->
+          <vertical>
+            <samples>60</samples>
+            <resolution>1</resolution>
+            <min_angle>-0.1221730476</min_angle>
+            <max_angle>0.9075712110</max_angle>
+          </vertical>
+        </scan>
+        <range>
+          <min>0.10</min>
+          <max>40.0</max>
+          <resolution>0.01</resolution>
+        </range>
+      </lidar>
+      <always_on>true</always_on>
+      <visualize>true</visualize>
+    </sensor>
+  </gazebo>
+  <!-- ================================ -->
+  <!-- RGB-D Camera Simulation          -->
+  <!-- ================================ -->
+  <gazebo reference="rgbd_camera_link">
+    <sensor name="rgbd_camera" type="rgbd_camera">
+      <gz_frame_id>rgbd_camera_link</gz_frame_id>
+      <camera>
+        <!-- 약 71.6 deg -->
+        <horizontal_fov>1.25</horizontal_fov>
+        <image>
+          <width>320</width>
+          <height>240</height>
+        </image>
+        <clip>
+          <near>0.10</near>
+          <far>5.0</far>
+        </clip>
+      </camera>
+      <always_on>true</always_on>
+      <!-- 현재 노트북 부하 고려 -->
+      <update_rate>15</update_rate>
+      <visualize>true</visualize>
+      <topic>rgbd_camera</topic>
+    </sensor>
+  </gazebo>
 </robot>

File: limbo/src/limbo_description/urdf/limbo.urdf.xacro (robot description, xacro)
@@ -2,13 +2,23 @@
 <robot xmlns:xacro="http://www.ros.org/wiki/xacro" name="Limbo">
   <!--
-    Limbo mobile robot - ROS 2 Jazzy / Gazebo Harmonic draft
+    Limbo mobile robot - ROS 2 Jazzy / Gazebo Harmonic
     Coordinate convention:
       +X = forward
       +Y = left
       +Z = up
-    Physical target envelope: 0.45 x 0.45 x 0.60 m
-    Nominal total mass used for simulation: 21.0 kg
-  -->
-  <!-- Geometry parameters -->
+    Updated exterior:
+      - plate.stl : main outer skeleton
+      - roof.stl  : low roof / MID-360 mounting structure
+    Mesh envelope (scale = 0.005):
+      plate: 0.45 x 0.45 m, approx. floor Z 0.0476 ~ 0.6105 m
+      roof : 0.45 x 0.45 m, approx. floor Z 0.6096 ~ 0.7103 m
+      MID-360 is centered at X=0, Y=0 on top of the roof.
+    Nominal total simulated mass remains 21.0 kg.
+  -->
+  <!-- ================================ -->
+  <!-- Geometry parameters              -->
+  <!-- ================================ -->
+  <!-- New CAD STL files are exported in the same coordinate system. -->
+  <xacro:property name="mesh_scale" value="0.005"/>
   <xacro:property name="wheel_radius" value="0.050"/>
   <xacro:property name="wheel_width" value="0.030"/>
@@ -29,19 +39,41 @@
   <xacro:property name="caster_wheel_z"
                   value="${caster_wheel_radius - caster_origin_z_global}"/>
-  <!--
-    Total caster mass remains 0.4 kg each.
-    Split between swivel assembly and wheel.
-  -->
+  <!-- Caster mass: 0.4 kg each -->
   <xacro:property name="caster_swivel_mass" value="0.10"/>
   <xacro:property name="caster_wheel_mass" value="0.30"/>
-  <!-- Nominal masses: total = 21.0 kg -->
-  <xacro:property name="body_mass" value="18.8"/>
+  <!--
+    Nominal masses: total = 21.0 kg
+      plate/body 18.6 + roof 0.2 + drive wheels 1.4 + casters 0.8 = 21.0 kg
+    roof_mass is provisional; replace it with the measured value later.
+  -->
+  <xacro:property name="body_mass" value="18.6"/>
+  <xacro:property name="roof_mass" value="0.2"/>
   <xacro:property name="wheel_mass" value="0.7"/>
-  <!-- Simplified body collision / inertia dimensions -->
+  <!-- Simplified collision / inertia dimensions for plate -->
   <xacro:property name="body_collision_x" value="0.45"/>
   <xacro:property name="body_collision_y" value="0.45"/>
-  <xacro:property name="body_collision_z" value="0.55"/>
-  <xacro:property name="body_com_z" value="0.275"/>
-  <!-- Inertia macros -->
+  <xacro:property name="body_collision_z" value="0.563"/>
+  <xacro:property name="body_com_z" value="0.279"/>
+  <!-- Simplified collision dimensions for the complete roof envelope. -->
+  <xacro:property name="roof_collision_x" value="0.45"/>
+  <xacro:property name="roof_collision_y" value="0.45"/>
+  <xacro:property name="roof_collision_z" value="0.101"/>
+  <!-- roof.stl bounds center, expressed relative to base_link/roof_link -->
+  <xacro:property name="roof_collision_center_z" value="0.60996"/>
+  <!--
+    roof.stl highest point is approx. 0.710301 m above the floor.
+    MID-360 measurement origin is placed 14.3 mm above the mounting surface.
+    Since base_link is 0.05 m above the floor:
+      0.710301 + 0.0143 - 0.05 = 0.674601 m
+    If you want the simulated ray origin exactly on the roof surface instead,
+    set mid360_measurement_origin_offset to 0.0.
+  -->
+  <xacro:property name="roof_top_z_global" value="0.710301"/>
+  <xacro:property name="mid360_measurement_origin_offset" value="0.0143"/>
+  <xacro:property name="mid360_z"
+                  value="${roof_top_z_global + mid360_measurement_origin_offset - base_link_height}"/>
+  <!-- ================================ -->
+  <!-- Inertia macros                   -->
+  <!-- ================================ -->
   <xacro:macro name="box_inertial" params="mass x y z origin_xyz">
     <inertial>
@@ -84,5 +116,7 @@
     </inertial>
   </xacro:macro>
-  <!-- Materials -->
+  <!-- ================================ -->
+  <!-- Materials                        -->
+  <!-- ================================ -->
   <material name="limbo_body_color">
     <color rgba="0.70 0.70 0.72 1.0"/>
@@ -91,5 +125,7 @@
     <color rgba="0.08 0.08 0.08 1.0"/>
   </material>
-  <!-- Base frames -->
+  <!-- ================================ -->
+  <!-- Base frames / plate              -->
+  <!-- ================================ -->
   <link name="base_footprint"/>
   <joint name="base_footprint_joint" type="fixed">
@@ -99,8 +135,14 @@
   </joint>
   <link name="base_link">
-    <visual name="body_visual">
+    <!--
+      Keep the existing 180-degree yaw correction so the CAD model's
+      intended front remains ROS +X.
+      plate.stl and roof.stl share the same CAD/world coordinate system.
+    -->
+    <visual name="plate_visual">
       <origin xyz="0 0 ${-base_link_height}" rpy="0 0 ${pi}"/>
       <geometry>
-        <mesh filename="package://limbo_description/meshes/body.stl"/>
+        <mesh filename="package://limbo_description/meshes/plate.stl"
+              scale="${mesh_scale} ${mesh_scale} ${mesh_scale}"/>
       </geometry>
       <material name="limbo_body_color"/>
@@ -119,5 +161,43 @@
       origin_xyz="0 0 ${body_com_z}"/>
   </link>
-  <!-- Drive wheels -->
+  <!-- ================================ -->
+  <!-- Roof                             -->
+  <!-- ================================ -->
+  <!--
+    roof.stl contains its CAD Z offset already, so roof_link shares the
+    same origin as base_link. The visual applies the same floor offset and
+    180-degree CAD yaw correction as plate.stl.
+  -->
+  <link name="roof_link">
+    <visual name="roof_visual">
+      <origin xyz="0 0 ${-base_link_height}" rpy="0 0 ${pi}"/>
+      <geometry>
+        <mesh filename="package://limbo_description/meshes/roof.stl"
+              scale="${mesh_scale} ${mesh_scale} ${mesh_scale}"/>
+      </geometry>
+      <material name="limbo_body_color"/>
+    </visual>
+    <!-- Conservative, low-cost collision approximation for simulation/self-filtering. -->
+    <collision name="roof_collision">
+      <origin xyz="0 0 ${roof_collision_center_z}" rpy="0 0 0"/>
+      <geometry>
+        <box size="${roof_collision_x} ${roof_collision_y} ${roof_collision_z}"/>
+      </geometry>
+    </collision>
+    <xacro:box_inertial
+      mass="${roof_mass}"
+      x="${roof_collision_x}"
+      y="${roof_collision_y}"
+      z="${roof_collision_z}"
+      origin_xyz="0 0 ${roof_collision_center_z}"/>
+  </link>
+  <joint name="roof_joint" type="fixed">
+    <parent link="base_link"/>
+    <child link="roof_link"/>
+    <origin xyz="0 0 0" rpy="0 0 0"/>
+  </joint>
+  <!-- ================================ -->
+  <!-- Drive wheels                     -->
+  <!-- ================================ -->
   <link name="left_wheel_link">
     <visual name="left_wheel_visual">
@@ -170,13 +250,7 @@
     <dynamics damping="0.05" friction="0.0"/>
   </joint>
-    <!-- ================================================== -->
-  <!-- Front caster                                       -->
-  <!-- ================================================== -->
-  <!--
-    The existing caster STL contains the complete caster
-    appearance. It is attached to the swivel link.
-    Collision / dynamics are modeled separately using
-    an invisible cylindrical caster wheel.
-  -->
+  <!-- ================================ -->
+  <!-- Front caster                     -->
+  <!-- ================================ -->
   <link name="front_caster_swivel_link">
     <visual name="front_caster_visual">
@@ -185,5 +259,4 @@
       </geometry>
     </visual>
-    <!-- Approximate inertia of caster bracket -->
     <xacro:box_inertial
       mass="${caster_swivel_mass}"
@@ -193,30 +266,16 @@
       origin_xyz="0 0 0"/>
   </link>
-  <!--
-    Swivel joint:
-    allows caster assembly to rotate freely around Z.
-  -->
   <joint name="front_caster_swivel_joint" type="continuous">
     <parent link="base_link"/>
     <child link="front_caster_swivel_link"/>
-    <origin xyz="${front_caster_x} 0 ${caster_joint_z}"
-            rpy="0 0 0"/>
+    <origin xyz="${front_caster_x} 0 ${caster_joint_z}" rpy="0 0 0"/>
     <axis xyz="0 0 1"/>
-    <!--
-      Small damping suppresses uncontrolled caster oscillation
-      while still allowing passive steering.
-    -->
-    <dynamics damping="0.10"
-              friction="0.01"/>
-  </joint>
-  <!-- Invisible physical caster wheel -->
+    <dynamics damping="0.10" friction="0.01"/>
+  </joint>
   <link name="front_caster_wheel_link">
     <collision name="front_caster_wheel_collision">
-      <origin xyz="0 0 0"
-              rpy="${pi/2.0} 0 0"/>
-      <geometry>
-        <cylinder
-          radius="${caster_wheel_radius}"
-          length="${caster_wheel_width}"/>
+      <origin xyz="0 0 0" rpy="${pi/2.0} 0 0"/>
+      <geometry>
+        <cylinder radius="${caster_wheel_radius}" length="${caster_wheel_width}"/>
       </geometry>
     </collision>
@@ -226,22 +285,14 @@
       width="${caster_wheel_width}"/>
   </link>
-  <!--
-    Wheel is offset behind the swivel axis.
-    This offset (caster trail) lets the caster naturally align
-    itself with the direction of travel.
-  -->
   <joint name="front_caster_wheel_joint" type="continuous">
     <parent link="front_caster_swivel_link"/>
     <child link="front_caster_wheel_link"/>
-    <origin
-      xyz="${-caster_trail} 0 ${caster_wheel_z}"
-      rpy="0 0 0"/>
+    <origin xyz="${-caster_trail} 0 ${caster_wheel_z}" rpy="0 0 0"/>
     <axis xyz="0 1 0"/>
-    <dynamics damping="0.02"
-              friction="0.0"/>
-  </joint>
-  <!-- ================================================== -->
-  <!-- Rear caster                                        -->
-  <!-- ================================================== -->
+    <dynamics damping="0.02" friction="0.0"/>
+  </joint>
+  <!-- ================================ -->
+  <!-- Rear caster                      -->
+  <!-- ================================ -->
   <link name="rear_caster_swivel_link">
     <visual name="rear_caster_visual">
@@ -260,18 +311,13 @@
     <parent link="base_link"/>
     <child link="rear_caster_swivel_link"/>
-    <origin xyz="${rear_caster_x} 0 ${caster_joint_z}"
-            rpy="0 0 0"/>
+    <origin xyz="${rear_caster_x} 0 ${caster_joint_z}" rpy="0 0 0"/>
     <axis xyz="0 0 1"/>
-    <dynamics damping="0.10"
-              friction="0.01"/>
+    <dynamics damping="0.10" friction="0.01"/>
   </joint>
   <link name="rear_caster_wheel_link">
     <collision name="rear_caster_wheel_collision">
-      <origin xyz="0 0 0"
-              rpy="${pi/2.0} 0 0"/>
-      <geometry>
-        <cylinder
-          radius="${caster_wheel_radius}"
-          length="${caster_wheel_width}"/>
+      <origin xyz="0 0 0" rpy="${pi/2.0} 0 0"/>
+      <geometry>
+        <cylinder radius="${caster_wheel_radius}" length="${caster_wheel_width}"/>
       </geometry>
     </collision>
@@ -284,25 +330,52 @@
     <parent link="rear_caster_swivel_link"/>
     <child link="rear_caster_wheel_link"/>
-    <origin
-      xyz="${-caster_trail} 0 ${caster_wheel_z}"
-      rpy="0 0 0"/>
+    <origin xyz="${-caster_trail} 0 ${caster_wheel_z}" rpy="0 0 0"/>
     <axis xyz="0 1 0"/>
-    <dynamics damping="0.02"
-              friction="0.0"/>
-  </joint>
-  <!-- ================================ -->
+    <dynamics damping="0.02" friction="0.0"/>
+  </joint>
   <!-- ================================ -->
   <!-- Livox MID-360                    -->
   <!-- ================================ -->
   <!--
-    MID-360 외형은 body.stl 안에 이미 포함되어 있음.
-    따라서 이 link는 센서의 좌표계(frame) 역할만 수행한다.
+    The MID-360 frame is no longer embedded in body.stl.
+    It is centered on the roof: X=0, Y=0.
+    Z is the sensor measurement origin above the roof mounting surface.
   -->
   <link name="mid360_link"/>
   <joint name="mid360_joint" type="fixed">
-    <parent link="base_link"/>
+    <parent link="roof_link"/>
     <child link="mid360_link"/>
-    <!-- body.stl에 모델링된 LiDAR 위치 -->
-    <origin xyz="0.19 0 0.59" rpy="0 0 0"/>
+    <origin xyz="0 0 ${mid360_z}" rpy="0 0 0"/>
+  </joint>
+  <!-- ================================ -->
+  <!-- RGB-D Camera                     -->
+  <!-- ================================ -->
+  <link name="rgbd_camera_link"/>
+  <joint name="rgbd_camera_joint" type="fixed">
+    <parent link="base_link"/>
+    <child link="rgbd_camera_link"/>
+    <!--
+      base_link는 바닥에서 0.05 m
+      camera 중심 목표 높이 약 0.30 m
+      따라서 base_link 기준 z = 0.25 m
+      x = +0.22 : 전방
+      pitch +10deg : 아래쪽을 향함
+    -->
+    <origin
+      xyz="0.22 0 0.40"
+      rpy="0 0.087266 0"/>
+  </joint>
+  <!-- ROS optical frame convention
+       X = right
+       Y = down
+       Z = forward
+  -->
+  <link name="rgbd_camera_optical_link"/>
+  <joint name="rgbd_camera_optical_joint" type="fixed">
+    <parent link="rgbd_camera_link"/>
+    <child link="rgbd_camera_optical_link"/>
+    <origin
+      xyz="0 0 0"
+      rpy="-1.570796 0 -1.570796"/>
   </joint>
   <xacro:include
