Commit message: 카메라를 0.7 m 아래 15°로 옮겨도 사람 검출·상자 costmap이 지금과 같다는 것을 12·15·18°로 확인하고, URDF·launch에 카메라 높이·피치 인자를 넣음 (67)
Co-Authored-By: Claude Fable 5.1 <noreply@anthropic.com>

File: limbo/src/limbo_description/urdf/limbo.urdf.xacro (robot description, xacro)
@@ -30,5 +30,10 @@
   <xacro:property name="camera_x" value="0.235"/>
   <xacro:property name="camera_y" value="0.1575"/>
-  <xacro:property name="camera_z" value="0.50"/>
+  <!-- 카메라 높이·아래로 기울인 각도(도). launch 인자 camera_z / camera_pitch_deg로 바꿀 수 있다 (센서 배치 실험용).
+       실물 마운트와 같은 값이어야 인식 좌표가 맞는다 -->
+  <xacro:arg name="camera_z" default="0.50"/>
+  <xacro:arg name="camera_pitch_deg" default="0"/>
+  <xacro:property name="camera_z" value="$(arg camera_z)"/>
+  <xacro:property name="camera_pitch" value="${radians($(arg camera_pitch_deg))}"/>
   <material name="body_gray"><color rgba="0.55 0.60 0.65 1.0"/></material>
   <material name="lid_gray"><color rgba="0.45 0.50 0.55 1.0"/></material>
@@ -162,5 +167,5 @@
     <parent link="base_link"/>
     <child link="rgbd_camera_link"/>
-    <origin xyz="${camera_x} ${camera_y} ${camera_z}" rpy="0 0 0"/>
+    <origin xyz="${camera_x} ${camera_y} ${camera_z}" rpy="0 ${camera_pitch} 0"/>
   </joint>
   <!-- ROS optical frame: X 오른쪽, Y 아래, Z 앞 -->

Commit message: 시뮬레이션에서 채택된 전역 STVL 3초·HumanLayer 치명 비용·prune_distance 2.5·카메라 0.7 m 15°·nav_recorder 지표와 새 문서를 ktj에 반영함 (31)
Co-Authored-By: Claude Fable 5.1 <noreply@anthropic.com>

File: limbo/src/limbo_description/urdf/limbo.urdf.xacro (robot description, xacro)
@@ -30,5 +30,12 @@
   <xacro:property name="camera_x" value="0.235"/>
   <xacro:property name="camera_y" value="0.1575"/>
-  <xacro:property name="camera_z" value="0.50"/>
+  <!-- 카메라 높이·아래로 기울인 각도(도). launch 인자 camera_z / camera_pitch_deg로 바꿀 수 있다.
+       2026-10-14 0.50 m 수평 → 0.70 m 아래 15°: 짧은 치마 밑단보다 높게 두어 올려다보는 구도를 없애고(개인정보),
+       근거리 바닥이 1.0 → 0.78 m 앞부터 보인다. 12·15·18° 시뮬레이션 비교에서 사람 검출·상자 costmap은 전과 같음.
+       실물 마운트와 같은 값이어야 인식 좌표가 맞는다. 기울인 깊이 카메라는 피치 오차 1°에 3 m 앞 바닥이 5 cm 떠 보이니 각도를 실측할 것 -->
+  <xacro:arg name="camera_z" default="0.70"/>
+  <xacro:arg name="camera_pitch_deg" default="15"/>
+  <xacro:property name="camera_z" value="$(arg camera_z)"/>
+  <xacro:property name="camera_pitch" value="${radians($(arg camera_pitch_deg))}"/>
   <material name="body_gray"><color rgba="0.55 0.60 0.65 1.0"/></material>
   <material name="lid_gray"><color rgba="0.45 0.50 0.55 1.0"/></material>
@@ -162,5 +169,5 @@
     <parent link="base_link"/>
     <child link="rgbd_camera_link"/>
-    <origin xyz="${camera_x} ${camera_y} ${camera_z}" rpy="0 0 0"/>
+    <origin xyz="${camera_x} ${camera_y} ${camera_z}" rpy="0 ${camera_pitch} 0"/>
   </joint>
   <!-- ROS optical frame: X 오른쪽, Y 아래, Z 앞 -->

Commit message: 저녁 채택분 반영: 사람이면 기다리기 BT·ToF 센서와 costmap·카메라 0.7 m 수평·MPPI 되돌이 처리·순찰 반복과 TF 출발·관제 일시정지 (32)
Co-Authored-By: Claude Fable 5.1 <noreply@anthropic.com>

File: limbo/src/limbo_description/urdf/limbo.urdf.xacro (robot description, xacro)
@@ -31,9 +31,10 @@
   <xacro:property name="camera_y" value="0.1575"/>
   <!-- 카메라 높이·아래로 기울인 각도(도). launch 인자 camera_z / camera_pitch_deg로 바꿀 수 있다.
-       2026-10-14 0.50 m 수평 → 0.70 m 아래 15°: 짧은 치마 밑단보다 높게 두어 올려다보는 구도를 없애고(개인정보),
-       근거리 바닥이 1.0 → 0.78 m 앞부터 보인다. 12·15·18° 시뮬레이션 비교에서 사람 검출·상자 costmap은 전과 같음.
-       실물 마운트와 같은 값이어야 인식 좌표가 맞는다. 기울인 깊이 카메라는 피치 오차 1°에 3 m 앞 바닥이 5 cm 떠 보이니 각도를 실측할 것 -->
+       2026-10-14 0.50 m 수평 → 0.70 m: 짧은 치마 밑단보다 높게 두어 올려다보는 구도를 없앤다(개인정보). 높이가 핵심, 각도는 부차.
+       각도는 0°: 15°는 근거리 바닥(0.78 m부터)이 보이지만 비스듬히 다가오는 손님의 상체가 잘려 전신 YOLO 검출이 19 % → 3 %로 떨어짐
+       (서브 PC 손님 장면 0/8/15° 각 3회). 근거리 바닥은 ToF(VL53L8CX)가 맡는다. 하반신 모델이 오면 0·8·15°를 다시 잰다(실물 브래킷은 각도 조절 가능하게).
+       실물 마운트와 같은 값이어야 인식 좌표가 맞는다 -->
   <xacro:arg name="camera_z" default="0.70"/>
-  <xacro:arg name="camera_pitch_deg" default="15"/>
+  <xacro:arg name="camera_pitch_deg" default="0"/>
   <xacro:property name="camera_z" value="$(arg camera_z)"/>
   <xacro:property name="camera_pitch" value="${radians($(arg camera_pitch_deg))}"/>
@@ -178,4 +179,15 @@
     <origin xyz="0 0 0" rpy="-1.570796 0 -1.570796"/>
   </joint>
+  <!-- ================================ -->
+  <!-- ToF 근접 센서 (VL53L5CX, 8x8)     -->
+  <!-- ================================ -->
+  <!-- 범퍼 높이 전면 중앙, 수평. 카메라가 못 보는 코앞(1.5 m 안)에 무언가 있는지만 본다 (R5).
+       차체 메시 앞면이 x 0.245라 그 바로 앞에 둔다 -->
+  <link name="tof_link"/>
+  <joint name="tof_joint" type="fixed">
+    <parent link="base_link"/>
+    <child link="tof_link"/>
+    <origin xyz="0.25 0 0.10" rpy="0 0 0"/>
+  </joint>
   <xacro:include filename="$(find limbo_description)/urdf/limbo.gazebo.xacro"/>
 </robot>

Commit message: 라이다 0.80 m(몸체 0.709)·default_server_timeout 100·벤치 도구 정리를 반영하고 주행 회귀 세트 결과를 기록함
Co-Authored-By: Claude Opus 5.5 <noreply@anthropic.com>

File: limbo/src/limbo_description/urdf/limbo.urdf.xacro (robot description, xacro)
@@ -13,5 +13,6 @@
   <!-- ================================ -->
   <xacro:property name="body_size" value="0.45"/>
-  <xacro:property name="body_top" value="0.835"/>
+  <!-- 몸체 윗면 높이. 2026-10-15 0.835 → 0.709: 뚜껑 위 MID-360이 바닥에서 0.80 m가 되게 몸체를 줄임(하드웨어 결정). 카메라는 0.70 m 그대로 -->
+  <xacro:property name="body_top" value="0.709"/>
   <xacro:property name="body_clearance" value="0.06"/>
   <xacro:property name="wheel_radius" value="0.075"/>
@@ -25,5 +26,5 @@
   <xacro:property name="lid_thickness" value="0.07"/>
   <xacro:property name="lid_open_max" value="1.9722220547535925"/>
-  <!-- MID-360: 뚜껑 위, 몸체 중심 위 바닥에서 약 0.926 m (경첩 높이 + 0.09094) -->
+  <!-- MID-360: 뚜껑 위, 몸체 중심 위 바닥에서 0.80 m (경첩 높이 0.709 + 0.09094) -->
   <xacro:property name="mid360_above_hinge" value="0.09094"/>
   <!-- OAK-D Lite: 앞면, 바닥에서 0.50 m, 중심에서 왼쪽 0.1575 m, 수평 (2026-10-12 결정) -->
@@ -59,5 +60,6 @@
     <visual>
       <geometry>
-        <mesh filename="package://limbo_description/meshes/v14/body.stl" scale="1 1 1"/>
+        <!-- 메시는 높이 0.835 m로 그려져 있어 body_top에 맞춰 z만 줄인다 (Gazebo 라이다는 시각 메시에 부딪히므로 메시가 높으면 자기 몸체를 본다, 2026-10-15) -->
+        <mesh filename="package://limbo_description/meshes/v14/body.stl" scale="1 1 ${body_top / 0.835}"/>
       </geometry>
       <material name="body_gray"/>

Commit message: 하드웨어 최종 치수에 맞춰 라이다를 바닥 0.70 m(몸체 높이 0.609)로, 카메라 기본 높이를 0.60 m로 낮췄다.
Co-Authored-By: Claude Opus 5.5 <noreply@anthropic.com>

File: limbo/src/limbo_description/urdf/limbo.urdf.xacro (robot description, xacro)
@@ -13,6 +13,6 @@
   <!-- ================================ -->
   <xacro:property name="body_size" value="0.45"/>
-  <!-- 몸체 윗면 높이. 2026-10-15 0.835 → 0.709: 뚜껑 위 MID-360이 바닥에서 0.80 m가 되게 몸체를 줄임(하드웨어 결정). 카메라는 0.70 m 그대로 -->
-  <xacro:property name="body_top" value="0.709"/>
+  <!-- 몸체 윗면 높이. 2026-10-15 0.835 → 0.609: 뚜껑 위 MID-360이 바닥에서 0.70 m가 되게 몸체를 줄임(하드웨어 최종 치수). 카메라는 0.60 m -->
+  <xacro:property name="body_top" value="0.609"/>
   <xacro:property name="body_clearance" value="0.06"/>
   <xacro:property name="wheel_radius" value="0.075"/>
@@ -26,15 +26,16 @@
   <xacro:property name="lid_thickness" value="0.07"/>
   <xacro:property name="lid_open_max" value="1.9722220547535925"/>
-  <!-- MID-360: 뚜껑 위, 몸체 중심 위 바닥에서 0.80 m (경첩 높이 0.709 + 0.09094) -->
+  <!-- MID-360: 뚜껑 위, 몸체 중심 위 바닥에서 0.70 m (경첩 높이 0.609 + 0.09094) -->
   <xacro:property name="mid360_above_hinge" value="0.09094"/>
-  <!-- OAK-D Lite: 앞면, 바닥에서 0.50 m, 중심에서 왼쪽 0.1575 m, 수평 (2026-10-12 결정) -->
+  <!-- OAK-D Lite: 앞면, 바닥에서 0.60 m(camera_z), 중심에서 왼쪽 0.1575 m, 수평 -->
   <xacro:property name="camera_x" value="0.235"/>
   <xacro:property name="camera_y" value="0.1575"/>
   <!-- 카메라 높이·아래로 기울인 각도(도). launch 인자 camera_z / camera_pitch_deg로 바꿀 수 있다.
        2026-10-14 0.50 m 수평 → 0.70 m: 짧은 치마 밑단보다 높게 두어 올려다보는 구도를 없앤다(개인정보). 높이가 핵심, 각도는 부차.
+       2026-10-15 하드웨어 최종 치수로 0.60 m(수평 그대로).
        각도는 0°: 15°는 근거리 바닥(0.78 m부터)이 보이지만 비스듬히 다가오는 손님의 상체가 잘려 전신 YOLO 검출이 19 % → 3 %로 떨어짐
        (서브 PC 손님 장면 0/8/15° 각 3회). 근거리 바닥은 ToF(VL53L8CX)가 맡는다. 하반신 모델이 오면 0·8·15°를 다시 잰다(실물 브래킷은 각도 조절 가능하게).
        실물 마운트와 같은 값이어야 인식 좌표가 맞는다 -->
-  <xacro:arg name="camera_z" default="0.70"/>
+  <xacro:arg name="camera_z" default="0.60"/>
   <xacro:arg name="camera_pitch_deg" default="0"/>
   <xacro:property name="camera_z" value="$(arg camera_z)"/>

Commit message: 하드웨어 최종 치수(라이다 0.70 m·카메라 0.60 m)와 default_server_timeout 100, 지도 작성 도구(make_map.sh·limbo_drive), 충장로 맛보기 생성기를 반영하고 문서를 고침 (33)
Co-Authored-By: Claude Opus 5.5 <noreply@anthropic.com>

File: limbo/src/limbo_description/urdf/limbo.urdf.xacro (robot description, xacro)
@@ -13,5 +13,6 @@
   <!-- ================================ -->
   <xacro:property name="body_size" value="0.45"/>
-  <xacro:property name="body_top" value="0.835"/>
+  <!-- 몸체 윗면 높이. 2026-10-15 0.835 → 0.609: 뚜껑 위 MID-360이 바닥에서 0.70 m가 되게 몸체를 줄임(하드웨어 최종 치수). 카메라는 0.60 m -->
+  <xacro:property name="body_top" value="0.609"/>
   <xacro:property name="body_clearance" value="0.06"/>
   <xacro:property name="wheel_radius" value="0.075"/>
@@ -25,15 +26,16 @@
   <xacro:property name="lid_thickness" value="0.07"/>
   <xacro:property name="lid_open_max" value="1.9722220547535925"/>
-  <!-- MID-360: 뚜껑 위, 몸체 중심 위 바닥에서 약 0.926 m (경첩 높이 + 0.09094) -->
+  <!-- MID-360: 뚜껑 위, 몸체 중심 위 바닥에서 0.70 m (경첩 높이 0.609 + 0.09094) -->
   <xacro:property name="mid360_above_hinge" value="0.09094"/>
-  <!-- OAK-D Lite: 앞면, 바닥에서 0.50 m, 중심에서 왼쪽 0.1575 m, 수평 (2026-10-12 결정) -->
+  <!-- OAK-D Lite: 앞면, 바닥에서 0.60 m(camera_z), 중심에서 왼쪽 0.1575 m, 수평 -->
   <xacro:property name="camera_x" value="0.235"/>
   <xacro:property name="camera_y" value="0.1575"/>
   <!-- 카메라 높이·아래로 기울인 각도(도). launch 인자 camera_z / camera_pitch_deg로 바꿀 수 있다.
        2026-10-14 0.50 m 수평 → 0.70 m: 짧은 치마 밑단보다 높게 두어 올려다보는 구도를 없앤다(개인정보). 높이가 핵심, 각도는 부차.
+       2026-10-15 하드웨어 최종 치수로 0.60 m(수평 그대로).
        각도는 0°: 15°는 근거리 바닥(0.78 m부터)이 보이지만 비스듬히 다가오는 손님의 상체가 잘려 전신 YOLO 검출이 19 % → 3 %로 떨어짐
        (손님 장면 0/8/15° 각 3회 시뮬레이션). 근거리 바닥은 ToF(VL53L8CX)가 맡는다. 하반신 모델이 오면 0·8·15°를 다시 잰다(실물 브래킷은 각도 조절 가능하게).
        실물 마운트와 같은 값이어야 인식 좌표가 맞는다 -->
-  <xacro:arg name="camera_z" default="0.70"/>
+  <xacro:arg name="camera_z" default="0.60"/>
   <xacro:arg name="camera_pitch_deg" default="0"/>
   <xacro:property name="camera_z" value="$(arg camera_z)"/>
@@ -59,5 +61,6 @@
     <visual>
       <geometry>
-        <mesh filename="package://limbo_description/meshes/v14/body.stl" scale="1 1 1"/>
+        <!-- 메시는 높이 0.835 m로 그려져 있어 body_top에 맞춰 z만 줄인다 (Gazebo 라이다는 시각 메시에 부딪히므로 메시가 높으면 자기 몸체를 본다, 2026-10-15) -->
+        <mesh filename="package://limbo_description/meshes/v14/body.stl" scale="1 1 ${body_top / 0.835}"/>
       </geometry>
       <material name="body_gray"/>
